Commit message: hardware interfaces stuff

File: sim/src/robo_courier/description/robot.urdf.xacro (robot description, xacro)
@@ -11,4 +11,4 @@
     </xacro:unless>
   <xacro:include filename="imu.xacro" />
-  <xacro:include filename="lidar.xacro" />
+  <!-- <xacro:include filename="lidar.xacro" />  -->
 </robot>

File: sim/src/robo_courier/description/robot_core.xacro (robot description, xacro)
@@ -121,5 +121,5 @@
         <child link="left_wheel_assembly"/>
         <origin xyz="${front_wheel_offset_x} ${wheel_offset_y} 0" rpy="0 0 0" />
-        <axis xyz="0 0 1" rpy="0 0 0" />
+        <axis xyz="0 0 -1" rpy="0 0 0" />
         <limit lower="-0.6" upper="0.6" velocity="1.0" effort="25"/>
     </joint>
@@ -182,9 +182,9 @@
     <material>Gazebo/White</material>
   </gazebo>
-    <joint name="right_wheel_hinge" type="revolute">
+   <joint name="right_wheel_hinge" type="revolute">
         <parent link="base_link"/>
         <child link="right_wheel_assembly"/>
         <origin xyz="${front_wheel_offset_x} -${wheel_offset_y} 0" rpy="0 0 0" />
-        <axis xyz="0 0 1" rpy="0 0 0" />
+        <axis xyz="0 0 -1" rpy="0 0 0" />  <!-- flipped sign -->
         <limit lower="-0.6" upper="0.6" velocity="1.0" effort="25"/>
     </joint>

File: sim/src/robo_courier/description/ros2_control.xacro (robot description, xacro)
@@ -11,5 +11,5 @@
         <param name="left_rear_wheel_joint">left_rear_wheel_joint</param>
         <param name="right_rear_wheel_joint">right_rear_wheel_joint</param>
-        <param name="loop_rate">30</param>
+        <param name="loop_rate">50</param>
         <param name="device">/dev/ttyUSB0</param>
         <param name="baud_rate">57600</param>
@@ -26,5 +26,4 @@
         <state_interface name="velocity"/>
       </joint>
-      <!-- Front Right Steering -->
       <joint name="right_wheel_hinge">
         <command_interface name="position">
@@ -35,5 +34,4 @@
         <state_interface name="velocity"/>
       </joint>
-      <!-- Rear Left Drive Wheel -->
       <joint name="left_rear_wheel_joint">
         <command_interface name="velocity">
@@ -44,5 +42,4 @@
         <state_interface name="velocity"/>
       </joint>
-      <!-- Rear Right Drive Wheel -->
       <joint name="right_rear_wheel_joint">
         <command_interface name="velocity">
