Commit message: ok does actually listen and print control, however ONLY when running ros2 run controller_manager ros2_control_node in a seperate temrinal

File: sim/src/robo_courier/description/ros2_control.xacro (robot description, xacro)
@@ -1,86 +1,103 @@
 <?xml version="1.0"?>
 <robot xmlns:xacro="http://www.ros.org/wiki/xacro">
-    <!-- <xacro:unless value="$(arg sim_mode)">
-        <ros2_control name="RealRobot" type="system">
-            <hardware>
-                <plugin>diffdrive_arduino/DiffDriveArduinoHardware</plugin>
-                <param name="left_wheel_name">left_wheel_joint</param>
-                <param name="right_wheel_name">right_wheel_joint</param>
-                <param name="loop_rate">30</param>
-                <param name="device">/dev/ttyUSB0</param>
-                <param name="baud_rate">57600</param>
-                <param name="timeout_ms">1000</param>
-                <param name="enc_counts_per_rev">3436</param>
-            </hardware>
-            <joint name="left_wheel_joint">
-                <command_interface name="velocity">
-                    <param name="min">-10</param>
-                    <param name="max">10</param>
-                </command_interface>
-                <state_interface name="position"/>
-                <state_interface name="velocity"/>
-            </joint>
-            <joint name="right_wheel_joint">
-                <command_interface name="velocity">
-                    <param name="min">-10</param>
-                    <param name="max">10</param>
-                </command_interface>
-                <state_interface name="position"/>
-                <state_interface name="velocity"/>
-            </joint>
-        </ros2_control>
-    </xacro:unless> -->
+  <!-- REAL HARDWARE INTERFACE -->
+  <xacro:unless value="$(arg sim_mode)">
+    <ros2_control name="RealRobot" type="system">
+      <hardware>
+        <plugin>ackdrive_arduino/AckDriveArduino</plugin>
+        <!-- Hardware parameters your C++ code reads -->
+        <param name="left_steer_joint">left_wheel_hinge</param>
+        <param name="right_steer_joint">right_wheel_hinge</param>
+        <param name="left_rear_wheel_joint">left_rear_wheel_joint</param>
+        <param name="right_rear_wheel_joint">right_rear_wheel_joint</param>
+        <param name="loop_rate">30</param>
+        <param name="device">/dev/ttyUSB0</param>
+        <param name="baud_rate">57600</param>
+        <param name="timeout">1000</param>
+        <param name="enc_counts_per_rev">3436</param>
+      </hardware>
+      <!-- Front Left Steering -->
+      <joint name="left_wheel_hinge">
+        <command_interface name="position">
+          <param name="min">-0.6</param>
+          <param name="max">0.6</param>
+        </command_interface>
+        <state_interface name="position"/>
+        <state_interface name="velocity"/>
+      </joint>
+      <!-- Front Right Steering -->
+      <joint name="right_wheel_hinge">
+        <command_interface name="position">
+          <param name="min">-0.6</param>
+          <param name="max">0.6</param>
+        </command_interface>
+        <state_interface name="position"/>
+        <state_interface name="velocity"/>
+      </joint>
+      <!-- Rear Left Drive Wheel -->
+      <joint name="left_rear_wheel_joint">
+        <command_interface name="velocity">
+          <param name="min">-10</param>
+          <param name="max">10</param>
+        </command_interface>
+        <state_interface name="position"/>
+        <state_interface name="velocity"/>
+      </joint>
+      <!-- Rear Right Drive Wheel -->
+      <joint name="right_rear_wheel_joint">
+        <command_interface name="velocity">
+          <param name="min">-10</param>
+          <param name="max">10</param>
+        </command_interface>
+        <state_interface name="position"/>
+        <state_interface name="velocity"/>
+      </joint>
+    </ros2_control>
+  </xacro:unless>
+  <!-- SIMULATION INTERFACE -->
+  <xacro:if value="$(arg sim_mode)">
     <ros2_control name="GazeboSystem" type="system">
-        <hardware>
-            <plugin>gazebo_ros2_control/GazeboSystem</plugin>
-        </hardware>
-        <joint name="left_wheel_hinge">
-            <command_interface name="velocity">
-                <param name="min">-1.0</param>
-                <param name="max">1.0</param>
-            </command_interface>
-            <command_interface name="position"/>
-            <state_interface name="velocity"/>
-            <state_interface name="position"/>
-        </joint>
-        <joint name="right_wheel_hinge">
-            <command_interface name="velocity">
-                <param name="min">-1.0</param>
-                <param name="max">1.0</param>
-            </command_interface>
-            <command_interface name="position"/>
-            <state_interface name="velocity"/>
-            <state_interface name="position"/>
-        </joint>
-        <joint name="left_rear_wheel_joint">
-            <command_interface name="velocity">
-                <param name="min">-10</param>
-                <param name="max">10</param>
-            </command_interface>
-            <state_interface name="velocity"/>
-            <state_interface name="position"/>
-        </joint>
-        <joint name="right_rear_wheel_joint">
-            <command_interface name="velocity">
-                <param name="min">-10</param>
-                <param name="max">10</param>
-            </command_interface>
-            <state_interface name="velocity"/>
-            <state_interface name="position"/>
-        </joint>
-        <joint name="front_left_rotate">
-            <!-- <command_interface name="position"/> -->
-            <state_interface name="position"/>
-        </joint>
-        <joint name="front_right_rotate">
-            <!-- <command_interface name="position"/> -->
-            <state_interface name="position"/>
-        </joint>
+      <hardware>
+        <plugin>gazebo_ros2_control/GazeboSystem</plugin>
+      </hardware>
+      <!-- Same joint definitions as above for Gazebo -->
+      <joint name="left_wheel_hinge">
+        <command_interface name="position">
+          <param name="min">-0.6</param>
+          <param name="max">0.6</param>
+        </command_interface>
+        <state_interface name="position"/>
+        <state_interface name="velocity"/>
+      </joint>
+      <joint name="right_wheel_hinge">
+        <command_interface name="position">
+          <param name="min">-0.6</param>
+          <param name="max">0.6</param>
+        </command_interface>
+        <state_interface name="position"/>
+        <state_interface name="velocity"/>
+      </joint>
+      <joint name="left_rear_wheel_joint">
+        <command_interface name="velocity">
+          <param name="min">-10</param>
+          <param name="max">10</param>
+        </command_interface>
+        <state_interface name="position"/>
+        <state_interface name="velocity"/>
+      </joint>
+      <joint name="right_rear_wheel_joint">
+        <command_interface name="velocity">
+          <param name="min">-10</param>
+          <param name="max">10</param>
+        </command_interface>
+        <state_interface name="position"/>
+        <state_interface name="velocity"/>
+      </joint>
     </ros2_control>
-    <gazebo>
-        <plugin name="gazebo_ros2_control" filename="libgazebo_ros2_control.so">
-            <parameters>$(find robo_courier)/config/my_controllers.yaml</parameters>
-            <parameters>$(find robo_courier)/config/gaz_ros2_ctl_use_sim.yaml</parameters>
-        </plugin>
-    </gazebo>
+  </xacro:if>
+  <gazebo>
+    <plugin name="gazebo_ros2_control" filename="libgazebo_ros2_control.so">
+      <parameters>$(find robo_courier)/config/my_controllers.yaml</parameters>
+    </plugin>
+  </gazebo>
 </robot>

Commit message: Add improvements to allow for mapping within the simulation. Autonomous navigation yet to be implemented

File: sim/src/robo_courier/description/ros2_control.xacro (robot description, xacro)
@@ -36,44 +36,30 @@
         </hardware>
         <joint name="left_wheel_hinge">
-            <command_interface name="velocity">
-                <param name="min">-1.0</param>
-                <param name="max">1.0</param>
-            </command_interface>
             <command_interface name="position"/>
+            <state_interface name="position"/>
             <state_interface name="velocity"/>
-            <state_interface name="position"/>
         </joint>
         <joint name="right_wheel_hinge">
-            <command_interface name="velocity">
-                <param name="min">-1.0</param>
-                <param name="max">1.0</param>
-            </command_interface>
             <command_interface name="position"/>
+            <state_interface name="position"/>
             <state_interface name="velocity"/>
-            <state_interface name="position"/>
         </joint>
         <joint name="left_rear_wheel_joint">
-            <command_interface name="velocity">
-                <param name="min">-10</param>
-                <param name="max">10</param>
-            </command_interface>
+            <command_interface name="velocity"/>
             <state_interface name="velocity"/>
             <state_interface name="position"/>
         </joint>
         <joint name="right_rear_wheel_joint">
-            <command_interface name="velocity">
-                <param name="min">-10</param>
-                <param name="max">10</param>
-            </command_interface>
+            <command_interface name="velocity"/>
             <state_interface name="velocity"/>
             <state_interface name="position"/>
         </joint>
         <joint name="front_left_rotate">
-            <!-- <command_interface name="position"/> -->
             <state_interface name="position"/>
+            <state_interface name="velocity"/>
         </joint>
         <joint name="front_right_rotate">
-            <!-- <command_interface name="position"/> -->
             <state_interface name="position"/>
+            <state_interface name="velocity"/>
         </joint>
     </ros2_control>
@@ -84,3 +70,39 @@
         </plugin>
     </gazebo>
+    <transmission name="left_front_steering_transmission">
+        <type>transmission_interface/SimpleTransmission</type>
+        <actuator name="left_front_steer_motor">
+            <mechanicalReduction>1.0</mechanicalReduction>
+        </actuator>
+        <joint name="left_wheel_hinge">
+            <hardwareInterface>hardware_interface/PositionCommand</hardwareInterface>
+        </joint>
+    </transmission>
+    <transmission name="right_front_steering_transmission">
+        <type>transmission_interface/SimpleTransmission</type>
+        <actuator name="right_front_steer_motor">
+            <mechanicalReduction>1.0</mechanicalReduction>
+        </actuator>
+        <joint name="right_wheel_hinge">
+            <hardwareInterface>hardware_interface/PositionCommand</hardwareInterface>
+        </joint>
+    </transmission>
+    <transmission name="left_rear_drive_transmission">
+        <type>transmission_interface/SimpleTransmission</type>
+        <actuator name="left_rear_drive_motor">
+            <mechanicalReduction>1.0</mechanicalReduction>
+        </actuator>
+        <joint name="left_rear_wheel_joint">
+            <hardwareInterface>hardware_interface/VelocityCommand</hardwareInterface>
+        </joint>
+    </transmission>
+    <transmission name="right_rear_drive_transmission">
+        <type>transmission_interface/SimpleTransmission</type>
+        <actuator name="right_rear_drive_motor">
+            <mechanicalReduction>1.0</mechanicalReduction>
+        </actuator>
+        <joint name="right_rear_wheel_joint">
+            <hardwareInterface>hardware_interface/VelocityCommand</hardwareInterface>
+        </joint>
+    </transmission>
 </robot>
